File: kiCad/PEE50_voltametrie.kicad_sch (KiCad schematic)
At the start: 52 parts, among them IC1 MIC5219-3.3YM5-TR, IC2 TPS7A2045PDBVR, IC3 TMUX1109PWR, IC5 ADS1113IDGSR, IC6 DAC80501MDGSR, IC7 LMP7702MA_NOPB, IC8 DS18B20+, J1 2201778-1, J2 USB_B_Micro, J4 Conn_02x03_Odd_Even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

Commit message: Version 2 kicad files
Before traces are added
Parts:
- J4: footprint Connector_PinHeader_2.54mm:PinHeader_2x03_P2.54mm_Vertical -> Connector_PinHeader_2.54mm:PinHeader_2x03_P2.54mm_Horizontal

Commit message: Version 3 kicad
Withoud 3.3V regulator not needed because of devkit
Parts:
- removed C2: 470p, Capacitor_SMD:C_0805_2012Metric_Pad1.18x1.45mm_HandSolder, symbol Device:C
- removed C3: 2.2u, Capacitor_SMD:C_0805_2012Metric_Pad1.18x1.45mm_HandSolder, symbol Device:C
- removed IC1: MIC5219-3.3YM5-TR, MIC5219-3.3YM5-TR:SOT95P280X145-5N, symbol MIC5219-3.3YM5-TR:MIC5219-3.3YM5-TR
- removed TP4: TestPoint, TestPoint:TestPoint_Pad_D1.0mm, symbol Connector:TestPoint
Connections:
- net 5V: now also U1.J2-19 (EXT_5V)
- net GND: now also U1.J2-14 (GND1), U1.J3-1 (GND3), U1.J3-7 (GND2)
- no-connect marks 38 -> 34

Commit message: layout aangepast
Parts:
- removed R13: 4k7, Resistor_SMD:R_0805_2012Metric_Pad1.20x1.40mm_HandSolder, symbol Device:R
Connections:
- net 3.3V: no longer C14.1, IC8.3 (VDD)
- net 4.5V: now also C14.1, IC8.3 (VDD), R8.2
- net temp: now also IC8.2 (DQ)
Other:
- moved on the sheet: R8

Commit message: SPI pin changes
Connections:
- net ChipSelect is gone; now on net CS1: IC6.7 (~{SYNC}/A0), R11.2, U1.J3-10 (IO5)
- net SDA2 is gone; now on net MOSI1: IC6.8 (SDIN/SDA), U1.J3-2 (IO23)
- net CS1: no longer J1.3 (CMD), R16.2, U1.J3-16 (IO15)
- net MOSI1: no longer J1.2 (CD/DAT3), R15.2, U1.J2-15 (IO13)
- net CLCK1 renamed SCK2
- net MISO1 renamed MISO2
- net SCL2 renamed SCK1
- new net CS2: J1.2 (CD/DAT3), R15.2, U1.J3-16 (IO15)
- new net MOSI2: J1.3 (CMD), R16.2, U1.J2-15 (IO13)
Other:
- moved on the sheet: C13
